Commit message: Update GEN3-6DOF_VISION_URDF_ARM_V01.urdf
matlab looks for end_effector_link to use

File: kortex_description/arms/gen3/6dof/urdf/GEN3-6DOF_VISION_URDF_ARM_V01.urdf (robot description, URDF)
Before this commit: robot GEN3-6DOF_VISION_URDF_ARM_V01, 8 links, 7 joints
Links:
- removed link EndEffector_Link
- added link end_effector_link, mass 0; collision mesh filename=package://kortex_description/arms/gen3/6dof/meshes/EndEffec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; visual mesh filename=package://kortex_description/arms/gen3/6dof/meshes/EndEffec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
